Commit message: fixed TF tree

File: april/model/camera.xacro (robot description, xacro)
@@ -5,5 +5,5 @@
     <!-- Pi constant -->
     <xacro:property name="pi_cam" value="3.14159265"/>
-        <link name="camera_link">
+        <link name="camera">
             <visual>
                 <geometry>
@@ -18,5 +18,5 @@
         <joint name="camera_joint" type="fixed">
             <parent link="${parent}"/>
-            <child link="camera_link"/>
+            <child link="camera"/>
             <xacro:insert_block name="origin"/>
         </joint>
@@ -24,5 +24,5 @@
         <link name="camera_optical_frame_link"></link>
         <joint name="camera_optical_frame_joint" type="fixed">
-            <parent link="camera_link"/>
+            <parent link="camera"/>
             <child link="camera_optical_frame_link"/>
             <origin xyz="0 0 0" rpy="${-pi_cam/2} 0 ${-pi_cam/2}"/>

File: april/model/robot.xacro (robot description, xacro)
@@ -55,5 +55,5 @@
 <!-- Body link of the robot-->
 <!-- allows us to render the box in gazebo -->
-<link name="body_link">
+<link name="base_link">
     <visual>
         <geometry>
@@ -74,5 +74,5 @@
 <!-- Back right wheel of the robot and the joint-->
  <joint name="wheel1_joint" type="continuous">
-    <parent link="body_link"/>
+    <parent link="base_link"/>
     <child link="wheel1_link"/>
     <!-- defined with respect to the coordinate frame of the parent link -->
@@ -101,5 +101,5 @@
 <!-- Back left wheel of the robot and the joint-->
  <joint name="wheel2_joint" type="continuous">
-    <parent link="body_link"/>
+    <parent link="base_link"/>
     <child link="wheel2_link"/>
     <!-- defined with respect to the coordinate frame of the parent link -->
@@ -128,5 +128,5 @@
 <!-- Front left wheel of the robot and the joint-->
  <joint name="wheel3_joint" type="continuous">
-    <parent link="body_link"/>
+    <parent link="base_link"/>
     <child link="wheel3_link"/>
     <!-- defined with respect to the coordinate frame of the parent link -->
@@ -155,5 +155,5 @@
 <!-- Front right wheel of the robot and the joint-->
  <joint name="wheel4_joint" type="continuous">
-    <parent link="body_link"/>
+    <parent link="base_link"/>
     <child link="wheel4_link"/>
     <!-- defined with respect to the coordinate frame of the parent link -->
@@ -182,5 +182,5 @@
 <!-- camera file -->
 <xacro:include filename="camera.xacro" />
-<xacro:logitech_C615 parent="body_link">
+<xacro:logitech_C615 parent="base_link">
     <origin xyz="${a/2} 0 ${c}" rpy="0 0 0"/>
 </xacro:logitech_C615>
