Commit message: Connected dummy map with NAV2

File: src/rdt_nav2_bringup/config/robot.xacro (robot description, xacro)
@@ -1,15 +1,9 @@
 <?xml version="1.0"?>
-<!-- Author: Andrea Gonzalez-->
 <robot name="rdt26_robot" xmlns:xacro="http://www.ros.org/wiki/xacro">
-<!-- Pi constant -->
 <xacro:property name="pi_const" value="3.14159265"/>
-<!-- Body dimensions-->
 <xacro:property name="a" value="1" />
 <xacro:property name="b" value="0.3" />
 <xacro:property name="c" value="0.6" />
-<!-- Wheel and caster dimensions -->
-<!-- Wheel and caster radius -->
 <xacro:property name="r" value="0.15" />
-<!-- Wheel width-->
 <xacro:property name="d" value="0.1" />
 <xacro:property name="s1" value="${b/2+r}" />
@@ -17,26 +11,15 @@
 <xacro:property name="s3" value="${2*r}" />
 <xacro:property name="s4" value="${c/2+d/2}" />
-<!-- Mass and Inertia-->
-<!-- Material density -->
-<!-- Body material density -->
 <xacro:property name="d1" value="2710.0" />
-<!-- Wheel material density -->
 <xacro:property name="d2" value="2710.0" />
-<!-- Robot body mass, wheel mass -->
-<!-- body -->
 <xacro:property name="m1" value="${d1*a*b*c}" />
-<!-- wheel -->
 <xacro:property name="m2" value="${d2*pi_const*r*r*d}" />
-<!-- Moments of interia of the robot body -->
 <xacro:property name="Ix_body" value="${(1/12)*m1*(b*b+c*c)}" />
 <xacro:property name="Iy_body" value="${(1/12)*m1*(a*a+b*b)}" />
 <xacro:property name="Iz_body" value="${(1/12)*m1*(a*a+c*c)}" />
-<!-- Moments of inertia of the wheel -->
 <xacro:property name="Iz_wheel" value="${0.5*m2*r*r}" />
 <xacro:property name="I_wheel" value="${(1.0/12.0)*m2*(3.0*r*r+d*d)}" />
-<!-- This macro defines the complete inertial section of the robot body -->
 <xacro:macro name="inertia_body">
     <inertial>
-    <!-- Displacement and orientation of the center of the mass-->
     <origin rpy="0 0 0" xyz="0 0 ${s1}" />
     <mass value="${m1}" />
@@ -44,5 +27,4 @@
     </inertial>
 </xacro:macro>
-<!-- This macro defines the complete inertial section of the wheel -->
 <xacro:macro name="inertia_wheel">
     <inertial>
@@ -52,10 +34,6 @@
     </inertial>
 </xacro:macro>
-<!-- Include addition files-->
-<!-- file that defines extra Gazebo options and motion control driver -->
 <xacro:include filename="$(find rdt_nav2_bringup)/config/robot.gazebo" />
 <xacro:include filename="$(find realsense2_description)/urdf/_d435.urdf.xacro"/>
-<!-- DEFINE LINKS, JOINTS -->
-<!-- Fictious link of the robot-->
 <link name="base_footprint"> </link>
 <joint name="body_link_joint" type="fixed">
@@ -63,6 +41,4 @@
     <child link="body_link"/>
 </joint>
-<!-- Body link of the robot-->
-<!-- allows us to render the box in gazebo -->
 <link name="body_link">
     <visual>
@@ -70,8 +46,6 @@
             <box size="${a} ${c} ${b}"/>
         </geometry>
-    <!-- Displacement and orientation of the geometric center of the link with respect to the link frame body_link_joint -->
     <origin rpy="0.0 0.0 0.0" xyz="0 0 ${s1}" />
     </visual>
-    <!-- how much collision space object/robot consumes -->
     <collision>
         <geometry>
@@ -82,13 +56,9 @@
     <xacro:inertia_body />
 </link>
-<!-- Back right wheel of the robot and the joint-->
- <joint name="wheel1_joint" type="continuous">
+<joint name="wheel1_joint" type="continuous">
     <parent link="body_link"/>
     <child link="wheel1_link"/>
-    <!-- defined with respect to the coordinate frame of the parent link -->
     <origin xyz="${-s2} ${-s4} ${r}" rpy="0.0 0.0 0.0" />
-    <!-- axis of rotation of the wheel -->
-    <axis xyz="0.0 1.0 0.0"/>
-    <!-- maximum torque -->
+    <axis xyz="0.0 1.0 0.0"/>
     <limit effort="50000" velocity="10"/>
     <dynamics damping="1.0" friction="1.0"/>
@@ -109,13 +79,9 @@
     <xacro:inertia_wheel />
 </link>
-<!-- Back left wheel of the robot and the joint-->
- <joint name="wheel2_joint" type="continuous">
+<joint name="wheel2_joint" type="continuous">
     <parent link="body_link"/>
     <child link="wheel2_link"/>
-    <!-- defined with respect to the coordinate frame of the parent link -->
     <origin xyz="${-s2} ${s4} ${r}" rpy="0.0 0.0 0.0" />
-    <!-- axis of rotation of the wheel -->
-    <axis xyz="0.0 1.0 0.0"/>
-    <!-- maximum torque -->
+    <axis xyz="0.0 1.0 0.0"/>
     <limit effort="50000" velocity="10"/>
     <dynamics damping="1.0" friction="1.0"/>
@@ -136,13 +102,9 @@
     <xacro:inertia_wheel />
 </link>
-<!-- Front left wheel of the robot and the joint-->
- <joint name="wheel3_joint" type="continuous">
+<joint name="wheel3_joint" type="continuous">
     <parent link="body_link"/>
     <child link="wheel3_link"/>
-    <!-- defined with respect to the coordinate frame of the parent link -->
     <origin xyz="${s3} ${s4} ${r}" rpy="0.0 0.0 0.0" />
-    <!-- axis of rotation of the wheel -->
-    <axis xyz="0.0 1.0 0.0"/>
-    <!-- maximum torque -->
+    <axis xyz="0.0 1.0 0.0"/>
     <limit effort="50000" velocity="10"/>
     <dynamics damping="1.0" friction="1.0"/>
@@ -163,13 +125,9 @@
     <xacro:inertia_wheel />
 </link>
-<!-- Front right wheel of the robot and the joint-->
- <joint name="wheel4_joint" type="continuous">
+<joint name="wheel4_joint" type="continuous">
     <parent link="body_link"/>
     <child link="wheel4_link"/>
-    <!-- defined with respect to the coordinate frame of the parent link -->
     <origin xyz="${s3} ${-s4} ${r}" rpy="0.0 0.0 0.0" />
-    <!-- axis of rotation of the wheel -->
-    <axis xyz="0.0 1.0 0.0"/>
-    <!-- maximum torque -->
+    <axis xyz="0.0 1.0 0.0"/>
     <limit effort="50000" velocity="10"/>
     <dynamics damping="1.0" friction="1.0"/>
@@ -242,6 +200,6 @@
     <origin xyz="0.4 0 ${s1 + 0.15}" rpy="0 0 0"/>
 </joint>
-<gazebo reference="laser_frame"> <sensor name="lidar" type="gpu_lidar">
-    <gz_frame_id>laser_frame</gz_frame_id> <topic>scan</topic>
+<gazebo reference="laser_frame"> <sensor name="laser_sensor" type="gpu_lidar">
+    <gz_frame_id>laser_frame</gz_frame_id> <topic>/scan</topic>
     <update_rate>10</update_rate>
     <ray>
