Commit message: updated robot xacro

File: src/pathplanning/pathplanning/robot.xacro (robot description, xacro)
@@ -1,219 +1,183 @@
 <?xml version="1.0"?>
-<!-- Author: Andrea Gonzalez-->
 <robot name="rdt26_robot" xmlns:xacro="http://www.ros.org/wiki/xacro">
-<!-- Pi constant -->
 <xacro:property name="pi_const" value="3.14159265"/>
-<!-- Body dimensions-->
-<xacro:property name="a" value="1" />
-<xacro:property name="b" value="0.3" />
-<xacro:property name="c" value="0.6" />
-<!-- Wheel and caster dimensions -->
-<!-- Wheel and caster radius -->
-<xacro:property name="r" value="0.15" />
-<!-- Wheel width-->
-<xacro:property name="d" value="0.1" />
-<xacro:property name="s1" value="${b/2+r}" />
-<xacro:property name="s2" value="${2*r}" />
-<xacro:property name="s3" value="${2*r}" />
-<xacro:property name="s4" value="${c/2+d/2}" />
-<!-- Mass and Inertia-->
+<!-- Real robot dimensions (metres) -->
+<xacro:property name="a" value="0.745" />   <!-- length -->
+<xacro:property name="b" value="0.608" />   <!-- width  -->
+<xacro:property name="c" value="0.660" />   <!-- height -->
+<!-- Wheel dimensions — measure and confirm these -->
+<xacro:property name="r" value="0.15" />    <!-- wheel radius -->
+<xacro:property name="d" value="0.1"  />    <!-- wheel width  -->
+<xacro:property name="s1" value="${c/2}"         />   <!-- body centre height -->
+<xacro:property name="s2" value="${a/2}"         />   <!-- wheel x offset (front/back) -->
+<xacro:property name="s3" value="${b/2 + d/2}"   />   <!-- wheel y offset (left/right) -->
 <!-- Material density -->
-<!-- Body material density -->
 <xacro:property name="d1" value="2710.0" />
-<!-- Wheel material density -->
 <xacro:property name="d2" value="2710.0" />
-<!-- Robot body mass, wheel mass -->
-<!-- body -->
+<!-- Mass -->
 <xacro:property name="m1" value="${d1*a*b*c}" />
-<!-- wheel -->
 <xacro:property name="m2" value="${d2*pi_const*r*r*d}" />
-<!-- Moments of interia of the robot body -->
+<!-- Inertia body -->
 <xacro:property name="Ix_body" value="${(1/12)*m1*(b*b+c*c)}" />
 <xacro:property name="Iy_body" value="${(1/12)*m1*(a*a+b*b)}" />
 <xacro:property name="Iz_body" value="${(1/12)*m1*(a*a+c*c)}" />
-<!-- Moments of inertia of the wheel -->
+<!-- Inertia wheel -->
 <xacro:property name="Iz_wheel" value="${0.5*m2*r*r}" />
-<xacro:property name="I_wheel" value="${(1.0/12.0)*m2*(3.0*r*r+d*d)}" />
-<!-- This macro defines the complete inertial section of the robot body -->
+<xacro:property name="I_wheel"  value="${(1.0/12.0)*m2*(3.0*r*r+d*d)}" />
 <xacro:macro name="inertia_body">
     <inertial>
-    <!-- Displacement and orientation of the center of the mass-->
-    <origin rpy="0 0 0" xyz="0 0 ${s1}" />
-    <mass value="${m1}" />
-    <inertia ixx="${Ix_body}" ixy="0.0" ixz="0.0" iyy="${Iy_body}" iyz="0" izz="${Iz_body}" />
+        <origin rpy="0 0 0" xyz="0 0 ${s1}"/>
+        <mass value="${m1}"/>
+        <inertia ixx="${Ix_body}" ixy="0" ixz="0"
+                                  iyy="${Iy_body}" iyz="0"
+                                                    izz="${Iz_body}"/>
     </inertial>
 </xacro:macro>
-<!-- This macro defines the complete inertial section of the wheel -->
 <xacro:macro name="inertia_wheel">
     <inertial>
-    <origin rpy="1.570795 0 0" xyz="0 0 0" />
-    <mass value="${m2}" />
-    <inertia ixx="${I_wheel}" ixy="0.0" ixz="0.0" iyy="${I_wheel}" iyz="0" izz="${Iz_wheel}" />
+        <origin rpy="1.570795 0 0" xyz="0 0 0"/>
+        <mass value="${m2}"/>
+        <inertia ixx="${I_wheel}" ixy="0" ixz="0"
+                                  iyy="${I_wheel}" iyz="0"
+                                                    izz="${Iz_wheel}"/>
     </inertial>
 </xacro:macro>
-<!-- Include addition files-->
-<!-- file that defines extra Gazebo options and motion control driver -->
-<xacro:include filename="$(find mobile_robot)/model/robot.gazebo" />
+<xacro:include filename="$(find mobile_robot)/model/robot.gazebo"/>
 <xacro:include filename="$(find realsense2_description)/urdf/_d435.urdf.xacro"/>
-<!-- DEFINE LINKS, JOINTS -->
-<!-- Fictious link of the robot-->
-<link name="base_footprint"> </link>
+<!-- ── Frames ─────────────────────────────────────────────────────────── -->
+<link name="base_footprint"/>
+<joint name="base_footprint_joint" type="fixed">
+    <parent link="base_footprint"/>
+    <child link="base_link"/>
+</joint>
+<!-- base_link: Nav2 + RTAB-Map reference frame, at ground centre -->
+<link name="base_link"/>
 <joint name="body_link_joint" type="fixed">
-    <parent link="base_footprint"/>
+    <parent link="base_link"/>
     <child link="body_link"/>
+    <origin xyz="0 0 0" rpy="0 0 0"/>
 </joint>
-<!-- Body link of the robot-->
-<!-- allows us to render the box in gazebo -->
 <link name="body_link">
     <visual>
         <geometry>
-            <box size="${a} ${c} ${b}"/>
+            <box size="${a} ${b} ${c}"/>
         </geometry>
-    <!-- Displacement and orientation of the geometric center of the link with respect to the link frame body_link_joint -->
-    <origin rpy="0.0 0.0 0.0" xyz="0 0 ${s1}" />
+        <origin rpy="0 0 0" xyz="0 0 ${s1}"/>
     </visual>
-    <!-- how much collision space object/robot consumes -->
     <collision>
         <geometry>
             <box size="${a} ${b} ${c}"/>
         </geometry>
-        <origin rpy="0.0 0.0 0.0" xyz="0 0 ${s1}" />
+        <origin rpy="0 0 0" xyz="0 0 ${s1}"/>
     </collision>
-    <xacro:inertia_body />
+    <xacro:inertia_body/>
 </link>
-<!-- Back right wheel of the robot and the joint-->
- <joint name="wheel1_joint" type="continuous">
-    <parent link="body_link"/>
+<!-- ── Wheels ─────────────────────────────────────────────────────────── -->
+<!-- Back right -->
+<joint name="wheel1_joint" type="continuous">
+    <parent link="base_link"/>
     <child link="wheel1_link"/>
-    <!-- defined with respect to the coordinate frame of the parent link -->
-    <origin xyz="${-s2} ${-s4} ${r}" rpy="0.0 0.0 0.0" />
-    <!-- axis of rotation of the wheel -->
-    <axis xyz="0.0 1.0 0.0"/>
-    <!-- maximum torque -->
+    <origin xyz="${-s2} ${-s3} ${r}" rpy="0 0 0"/>
+    <axis xyz="0 1 0"/>
     <limit effort="50000" velocity="10"/>
     <dynamics damping="1.0" friction="1.0"/>
- </joint>
- <link name="wheel1_link">
+</joint>
+<link name="wheel1_link">
     <visual>
-        <origin xyz="0.0 0.0 0.0" rpy="1.570795 0.0 0.0"/>
-        <geometry>
-            <cylinder radius="${r}" length="${d}"/>
-        </geometry>
+        <origin xyz="0 0 0" rpy="1.570795 0 0"/>
+        <geometry><cylinder radius="${r}" length="${d}"/></geometry>
     </visual>
     <collision>
-        <origin xyz="0.0 0.0 0.0" rpy="1.570795 0.0 0.0"/>
-        <geometry>
-            <cylinder radius="${r}" length="${d}"/>
-        </geometry>
+        <origin xyz="0 0 0" rpy="1.570795 0 0"/>
+        <geometry><cylinder radius="${r}" length="${d}"/></geometry>
     </collision>
-    <xacro:inertia_wheel />
+    <xacro:inertia_wheel/>
 </link>
-<!-- Back left wheel of the robot and the joint-->
- <joint name="wheel2_joint" type="continuous">
-    <parent link="body_link"/>
+<!-- Back left -->
+<joint name="wheel2_joint" type="continuous">
+    <parent link="base_link"/>
     <child link="wheel2_link"/>
-    <!-- defined with respect to the coordinate frame of the parent link -->
-    <origin xyz="${-s2} ${s4} ${r}" rpy="0.0 0.0 0.0" />
-    <!-- axis of rotation of the wheel -->
-    <axis xyz="0.0 1.0 0.0"/>
-    <!-- maximum torque -->
+    <origin xyz="${-s2} ${s3} ${r}" rpy="0 0 0"/>
+    <axis xyz="0 1 0"/>
     <limit effort="50000" velocity="10"/>
     <dynamics damping="1.0" friction="1.0"/>
- </joint>
- <link name="wheel2_link">
+</joint>
+<link name="wheel2_link">
     <visual>
-        <origin xyz="0.0 0.0 0.0" rpy="1.570795 0.0 0.0"/>
-        <geometry>
-            <cylinder radius="${r}" length="${d}"/>
-        </geometry>
+        <origin xyz="0 0 0" rpy="1.570795 0 0"/>
+        <geometry><cylinder radius="${r}" length="${d}"/></geometry>
     </visual>
     <collision>
-        <origin xyz="0.0 0.0 0.0" rpy="1.570795 0.0 0.0"/>
-        <geometry>
-            <cylinder radius="${r}" length="${d}"/>
-        </geometry>
+        <origin xyz="0 0 0" rpy="1.570795 0 0"/>
+        <geometry><cylinder radius="${r}" length="${d}"/></geometry>
     </collision>
-    <xacro:inertia_wheel />
+    <xacro:inertia_wheel/>
 </link>
-<!-- Front left wheel of the robot and the joint-->
- <joint name="wheel3_joint" type="continuous">
-    <parent link="body_link"/>
+<!-- Front left -->
+<joint name="wheel3_joint" type="continuous">
+    <parent link="base_link"/>
     <child link="wheel3_link"/>
-    <!-- defined with respect to the coordinate frame of the parent link -->
-    <origin xyz="${s3} ${s4} ${r}" rpy="0.0 0.0 0.0" />
-    <!-- axis of rotation of the wheel -->
-    <axis xyz="0.0 1.0 0.0"/>
-    <!-- maximum torque -->
+    <origin xyz="${s2} ${s3} ${r}" rpy="0 0 0"/>
+    <axis xyz="0 1 0"/>
     <limit effort="50000" velocity="10"/>
     <dynamics damping="1.0" friction="1.0"/>
- </joint>
- <link name="wheel3_link">
+</joint>
+<link name="wheel3_link">
     <visual>
-        <origin xyz="0.0 0.0 0.0" rpy="1.570795 0.0 0.0"/>
-        <geometry>
-            <cylinder radius="${r}" length="${d}"/>
-        </geometry>
+        <origin xyz="0 0 0" rpy="1.570795 0 0"/>
+        <geometry><cylinder radius="${r}" length="${d}"/></geometry>
     </visual>
     <collision>
-        <origin xyz="0.0 0.0 0.0" rpy="1.570795 0.0 0.0"/>
-        <geometry>
-            <cylinder radius="${r}" length="${d}"/>
-        </geometry>
+        <origin xyz="0 0 0" rpy="1.570795 0 0"/>
+        <geometry><cylinder radius="${r}" length="${d}"/></geometry>
     </collision>
-    <xacro:inertia_wheel />
+    <xacro:inertia_wheel/>
 </link>
-<!-- Front right wheel of the robot and the joint-->
- <joint name="wheel4_joint" type="continuous">
-    <parent link="body_link"/>
+<!-- Front right -->
+<joint name="wheel4_joint" type="continuous">
+    <parent link="base_link"/>
     <child link="wheel4_link"/>
-    <!-- defined with respect to the coordinate frame of the parent link -->
-    <origin xyz="${s3} ${-s4} ${r}" rpy="0.0 0.0 0.0" />
-    <!-- axis of rotation of the wheel -->
-    <axis xyz="0.0 1.0 0.0"/>
-    <!-- maximum torque -->
+    <origin xyz="${s2} ${-s3} ${r}" rpy="0 0 0"/>
+    <axis xyz="0 1 0"/>
     <limit effort="50000" velocity="10"/>
     <dynamics damping="1.0" friction="1.0"/>
- </joint>
- <link name="wheel4_link">
+</joint>
+<link name="wheel4_link">
     <visual>
-        <origin xyz="0.0 0.0 0.0" rpy="1.570795 0.0 0.0"/>
-        <geometry>
-            <cylinder radius="${r}" length="${d}"/>
-        </geometry>
+        <origin xyz="0 0 0" rpy="1.570795 0 0"/>
+        <geometry><cylinder radius="${r}" length="${d}"/></geometry>
     </visual>
     <collision>
-        <origin xyz="0.0 0.0 0.0" rpy="1.570795 0.0 0.0"/>
-        <geometry>
-            <cylinder radius="${r}" length="${d}"/>
-        </geometry>
+        <origin xyz="0 0 0" rpy="1.570795 0 0"/>
+        <geometry><cylinder radius="${r}" length="${d}"/></geometry>
     </collision>
-    <xacro:inertia_wheel />
+    <xacro:inertia_wheel/>
 </link>
-<xacro:sensor_d435 parent="body_link" name="camera" use_nominal_extrinsics="true">
-    <origin xyz="0.5 0 0.3" rpy="0 0 0"/>
+<!-- ── RealSense D435 ──────────────────────────────────────────────────── -->
+<!-- mounted at front face centre, ~33cm off ground -->
+<xacro:sensor_d435 parent="base_link" name="camera" use_nominal_extrinsics="true">
+    <origin xyz="0.37 0.0 0.33" rpy="0 0 0"/>
 </xacro:sensor_d435>
 <gazebo reference="camera_link">
-  <sensor name="realsense_d435" type="rgbd_camera">
-    <topic>realsense</topic> <camera>
-      <horizontal_fov>1.047</horizontal_fov>
-      <image>
-        <width>640</width>
-        <height>480</height>
-        <format>R8G8B8</format>
-      </image>
-      <clip>
-        <near>0.1</near>
-        <far>100</far>
-      </clip>
-      <noise>
-          <type>gaussian</type>
-          <mean>0.0</mean>
-          <stddev>0.007</stddev>
-      </noise>
-    </camera>
-    <always_on>1</always_on>
-    <update_rate>30</update_rate>
-    <visualize>true</visualize>
-  </sensor>
+    <sensor name="realsense_d435" type="rgbd_camera">
+        <topic>realsense</topic>
+        <camera>
+            <horizontal_fov>1.047</horizontal_fov>
+            <image>
+                <width>640</width>
+                <height>480</height>
+                <format>R8G8B8</format>
+            </image>
+            <clip><near>0.1</near><far>100</far></clip>
+            <noise>
+                <type>gaussian</type>
+                <mean>0.0</mean>
+                <stddev>0.007</stddev>
+            </noise>
+        </camera>
+        <always_on>1</always_on>
+        <update_rate>30</update_rate>
+        <visualize>true</visualize>
+    </sensor>
 </gazebo>
 </robot>
