Commit message: removed extra files and renames some pkgs

File: src/nyurdt_navigation/config/robot.xacro (robot description, xacro)
@@ -34,5 +34,5 @@
     </inertial>
 </xacro:macro>
-<xacro:include filename="$(find rdt_nav2_bringup)/config/robot.gazebo" />
+<xacro:include filename="$(find nyurdt_navigation)/config/robot.gazebo" />
 <xacro:include filename="$(find realsense2_description)/urdf/_d435.urdf.xacro"/>
 <link name="base_footprint"> </link>
@@ -175,48 +175,3 @@
   </sensor>
 </gazebo>
-<link name="laser_frame">
-    <visual>
-        <geometry>
-            <cylinder radius="0.05" length="0.04"/>
-        </geometry>
-        <material name="black">
-            <color rgba="0 0 0 1"/>
-        </material>
-    </visual>
-    <collision>
-        <geometry>
-            <cylinder radius="0.05" length="0.04"/>
-        </geometry>
-    </collision>
-    <inertial>
-        <mass value="0.1" />
-        <origin xyz="0 0 0" rpy="0 0 0"/>
-        <inertia ixx="0.0001" ixy="0" ixz="0" iyy="0.0001" iyz="0" izz="0.0001" />
-    </inertial>
-</link>
-<joint name="laser_joint" type="fixed">
-    <parent link="body_link"/>
-    <child link="laser_frame"/>
-    <origin xyz="0.4 0 ${s1 + 0.15}" rpy="0 0 0"/>
-</joint>
-<gazebo reference="laser_frame"> <sensor name="laser_sensor" type="gpu_lidar">
-    <gz_frame_id>laser_frame</gz_frame_id> <topic>/scan</topic>
-    <update_rate>10</update_rate>
-    <ray>
-      <scan>
-        <horizontal>
-          <samples>360</samples>
-          <resolution>1</resolution>
-          <min_angle>-3.14</min_angle>
-          <max_angle>3.14</max_angle>
-        </horizontal>
-      </scan>
-      <range>
-        <min>0.1</min>
-        <max>12.0</max>
-      </range>
-    </ray>
-    <visualize>true</visualize>
-  </sensor>
-</gazebo>
 </robot>
