Commit message: multiple camera integration wip

File: src/nyurdt_localization/model/camera.xacro (robot description, xacro)
@@ -2,12 +2,12 @@
 <!-- Author: Mandy Wang-->
 <robot xmlns:xacro="http://www.ros.org/wiki/xacro">
-    <xacro:macro name="logitech_C615" params="parent *origin">
+    <xacro:macro name="camera" params="parent pos size_x size_y size_z *origin">
     <!-- Pi constant -->
     <xacro:property name="pi_cam" value="3.14159265"/>
-        <link name="camera">
+        <link name="${pos}_camera">
             <visual>
                 <geometry>
                     <!-- logitech C615 -->
-                    <box size="0.017 0.07 0.04"/>
+                    <box size="${size_x} ${size_y} ${size_z}"/>
                 </geometry>
                 <material name="black">
@@ -16,14 +16,14 @@
             </visual>
         </link>
-        <joint name="camera_joint" type="fixed">
+        <joint name="${pos}_camera_joint" type="fixed">
             <parent link="${parent}"/>
-            <child link="camera"/>
+            <child link="${pos}_camera"/>
             <xacro:insert_block name="origin"/>
         </joint>
         <!--vision frame used by image and tf topics-->
-        <link name="camera_optical_frame_link"></link>
-        <joint name="camera_optical_frame_joint" type="fixed">
-            <parent link="camera"/>
-            <child link="camera_optical_frame_link"/>
+        <link name="${pos}_camera_optical_frame_link"></link>
+        <joint name="${pos}_camera_optical_frame_joint" type="fixed">
+            <parent link="${pos}_camera"/>
+            <child link="${pos}_camera_optical_frame_link"/>
             <origin xyz="0 0 0" rpy="${-pi_cam/2} 0 ${-pi_cam/2}"/>
         </joint>

File: src/nyurdt_localization/model/robot.xacro (robot description, xacro)
@@ -182,6 +182,12 @@
 <!-- camera file -->
 <xacro:include filename="camera.xacro" />
-<xacro:logitech_C615 parent="base_link">
+<xacro:property name="x" value=".017"/>
+<xacro:property name="y" value=".07"/>
+<xacro:property name="z" value=".04"/>
+<xacro:camera parent="base_link" pos="front" size_x="${x}" size_y="${y}" size_z="${z}">
     <origin xyz="${a/2} 0 ${c}" rpy="0 0 0"/>
-</xacro:logitech_C615>
+</xacro:camera>
+<xacro:camera parent="base_link" pos="right" size_x="${x}" size_y="${y}" size_z="${z}">
+    <origin xyz="${a/2} 0 ${c}" rpy="0 0 0"/>
+</xacro:camera>
 </robot>

Commit message: changed apriltag pose numbers, updated cam offsets, and updated robot origin

File: src/nyurdt_localization/model/camera.xacro (robot description, xacro)
@@ -8,5 +8,4 @@
             <visual>
                 <geometry>
-                    <!-- logitech C615 -->
                     <box size="${size_x} ${size_y} ${size_z}"/>
                 </geometry>

File: src/nyurdt_localization/model/robot1.xacro (robot description, xacro)
@@ -3,5 +3,5 @@
 <link name="base_link">
 <visual>
-    <origin xyz="0 0 0" rpy="0 0 0"/>
+    <origin xyz="-0.21971 -0.18098 0" rpy="0 0 0"/>
     <geometry>
     <mesh filename="package://nyurdt_localization/model/robot.stl"
@@ -10,7 +10,7 @@
 </visual>
 <collision>
-    <origin xyz="0 0 0" rpy="0 0 0"/>
+    <origin xyz="-0.21971 -0.18098 0" rpy="0 0 0"/>
     <geometry>
-    <box size="0.7 0.5 0.3"/>
+    <box size="0.74784 0.60788 0.5"/>
     </geometry>
 </collision>
@@ -23,3 +23,25 @@
 </inertial>
 </link>
+<!-- camera file -->
+<xacro:include filename="camera.xacro" />
+<xacro:property name="x" value=".017"/>
+<xacro:property name="y" value=".07"/>
+<xacro:property name="z" value=".04"/>
+<xacro:camera parent="base_link" pos="left" size_x="${x}" size_y="${y}" size_z="${z}">
+    <origin xyz="0.00792 0.195 0.26" rpy="0 0 0"/>
+</xacro:camera>
+<xacro:camera parent="base_link" pos="right" size_x="${x}" size_y="${y}" size_z="${z}">
+    <origin xyz="0.00792 -0.195 0.26" rpy="0 0 0"/>
+</xacro:camera>
+<!-- camera file -->
+<xacro:include filename="camera.xacro" />
+<xacro:property name="x" value=".037"/>
+<xacro:property name="y" value=".037"/>
+<xacro:property name="z" value=".04"/>
+<xacro:camera parent="base_link" pos="front" size_x="${x}" size_y="${y}" size_z="${z}">
+    <origin xyz="0 0 0" rpy="0 0 0"/>
+</xacro:camera>
+<xacro:camera parent="base_link" pos="back" size_x="${x}" size_y="${y}" size_z="${z}">
+    <origin xyz="0 0 0" rpy="0 0 0"/>
+</xacro:camera>
 </robot>
