Commit message: Apriltag (#54)
* combining camera sensor launch

* [April] modified camera resolution

* deleted extra files

* pose publishing based on apriltag_ros

* recalibration wip

* recalibration wip

* 1600x896 test

* [April] modified apriltag_tf.py and logitech yaml

* multiple camera integration wip

* multiple camera integration wip

* multiple camera integration wip

* updated tags and verified multiple cameras launching

* calibration wip

* calibration wip

* calibration wip

* calibration wip

* added robot model

* tag and cam offset wip

* [Apriltag] updated tag pose in map

* wip

* coney testing numbers

Updated camera origin positions to (0, 0, 0) for both front and right cameras.

* changed apriltag pose numbers, updated cam offsets, and updated robot origin

* added cams (missing index and front cam pos)

---------

Co-authored-by: MdyWg <mdywg16@gmail.com>
Co-authored-by: chasemike <michaelstevencarcamo@gmail.com>
Co-authored-by: Andrea Gonzalez <andrea7308.github.io>
Co-authored-by: calistaroldan <clr9232@nyu.edu>

File: src/nyurdt_description/urdf/camera.xacro (robot description, xacro)
@@ -2,12 +2,11 @@
 <!-- Author: Mandy Wang-->
 <robot xmlns:xacro="http://www.ros.org/wiki/xacro">
-    <xacro:macro name="logitech_C615" params="parent *origin">
+    <xacro:macro name="camera" params="parent pos size_x size_y size_z *origin">
     <!-- Pi constant -->
     <xacro:property name="pi_cam" value="3.14159265"/>
-        <link name="camera">
+        <link name="${pos}_camera">
             <visual>
                 <geometry>
-                    <!-- logitech C615 -->
-                    <box size="0.017 0.07 0.04"/>
+                    <box size="${size_x} ${size_y} ${size_z}"/>
                 </geometry>
                 <material name="black">
@@ -16,14 +15,14 @@
             </visual>
         </link>
-        <joint name="camera_joint" type="fixed">
+        <joint name="${pos}_camera_joint" type="fixed">
             <parent link="${parent}"/>
-            <child link="camera"/>
+            <child link="${pos}_camera"/>
             <xacro:insert_block name="origin"/>
         </joint>
         <!--vision frame used by image and tf topics-->
-        <link name="camera_optical_frame_link"></link>
-        <joint name="camera_optical_frame_joint" type="fixed">
-            <parent link="camera"/>
-            <child link="camera_optical_frame_link"/>
+        <link name="${pos}_camera_optical_frame_link"></link>
+        <joint name="${pos}_camera_optical_frame_joint" type="fixed">
+            <parent link="${pos}_camera"/>
+            <child link="${pos}_camera_optical_frame_link"/>
             <origin xyz="0 0 0" rpy="${-pi_cam/2} 0 ${-pi_cam/2}"/>
         </joint>

File: src/nyurdt_description/urdf/robot.xacro (robot description, xacro)
@@ -176,3 +176,26 @@
     </sensor>
 </gazebo>
+<!-- ── Logitech C615 ──────────────────────────────────────────────────── -->
+<xacro:include filename="camera.xacro" />
+<xacro:property name="x" value=".017"/>
+<xacro:property name="y" value=".07"/>
+<xacro:property name="z" value=".04"/>
+<!-- need numbers -->
+<xacro:camera parent="base_link" pos="front" size_x="${x}" size_y="${y}" size_z="${z}">
+    <origin xyz="0 0 0" rpy="0 0 0"/>
+</xacro:camera>
+<xacro:camera parent="base_link" pos="back" size_x="${x}" size_y="${y}" size_z="${z}">
+    <origin xyz="-.2799208 -.195 .45" rpy="0 0 -${pi_const}"/>
+</xacro:camera>
+<!-- ── Innomaker ──────────────────────────────────────────────────── -->
+<xacro:include filename="camera.xacro" />
+<xacro:property name="x" value=".037"/>
+<xacro:property name="y" value=".037"/>
+<xacro:property name="z" value=".04"/>
+<xacro:camera parent="base_link" pos="right" size_x="${x}" size_y="${y}" size_z="${z}">
+    <origin xyz="0.00792 -0.195 0.45" rpy="0 0 -1.57"/>
+</xacro:camera>
+<xacro:camera parent="base_link" pos="left" size_x="${x}" size_y="${y}" size_z="${z}">
+    <origin xyz="0.00792 0.195 0.45" rpy="0 0 1.57"/>
+</xacro:camera>
 </robot>

Commit message: -

File: src/nyurdt_description/urdf/camera.xacro (robot description, xacro)
@@ -27,4 +27,34 @@
             <origin xyz="0 0 0" rpy="${-pi_cam/2} 0 ${-pi_cam/2}"/>
         </joint>
+        <!-- Simulated camera using rgbd_camera (works with ogre render engine).
+             body_link is transparent in robot.gazebo so cameras inside the robot
+             body can see through it and render images correctly. -->
+        <gazebo reference="${pos}_camera">
+            <sensor name="${pos}_cam" type="rgbd_camera">
+                <topic>${pos}_cam</topic>
+                <camera>
+                    <horizontal_fov>1.047</horizontal_fov>
+                    <image>
+                        <width>320</width>
+                        <height>240</height>
+                        <format>R8G8B8</format>
+                    </image>
+                    <clip>
+                        <near>0.1</near>
+                        <far>8.0</far>
+                    </clip>
+                    <depth_camera>
+                        <output>depths</output>
+                        <clip>
+                            <near>0.1</near>
+                            <far>8.0</far>
+                        </clip>
+                    </depth_camera>
+                </camera>
+                <always_on>1</always_on>
+                <update_rate>5</update_rate>
+                <visualize>false</visualize>
+            </sensor>
+        </gazebo>
     </xacro:macro>
 </robot>

File: src/nyurdt_description/urdf/robot.xacro (robot description, xacro)
@@ -152,7 +152,15 @@
 <!-- mounted at front face centre, ~33cm off ground -->
 <xacro:sensor_d435 parent="base_link" name="camera" use_nominal_extrinsics="true">
-    <origin xyz="0.37 0.0 0.33" rpy="0 0.767945 0"/>
+    <origin xyz="0.37 0.0 0.78" rpy="0 0.767945 0"/>
 </xacro:sensor_d435>
 <gazebo reference="camera_link">
+    <!--
+      Simulated RealSense D435 (rgbd_camera).
+      Gazebo publishes on topic prefix "realsense":
+        /realsense/image          → color image (bridged to /camera/camera/color/image_raw)
+        /realsense/depth_image    → depth image (bridged to /camera/camera/depth/image_rect_raw)
+        /realsense/camera_info    → camera info (bridged to /camera/camera/color/camera_info)
+        /realsense/points         → point cloud (bridged to /camera/camera/depth/points)
+    -->
     <sensor name="realsense_d435" type="rgbd_camera">
         <topic>realsense</topic>
@@ -160,18 +168,26 @@
             <horizontal_fov>1.047</horizontal_fov>
             <image>
-                <width>640</width>
-                <height>480</height>
+                <width>424</width>
+                <height>240</height>
                 <format>R8G8B8</format>
             </image>
-            <clip><near>0.1</near><far>100</far></clip>
+            <depth_camera>
+                <output>depths</output>
+                <clip>
+                    <near>0.1</near>
+                    <far>5.0</far>
+                </clip>
+            </depth_camera>
+            <clip><near>0.1</near><far>5.0</far></clip>
             <noise>
                 <type>gaussian</type>
                 <mean>0.0</mean>
-                <stddev>0.007</stddev>
+                <stddev>0.005</stddev>
             </noise>
         </camera>
         <always_on>1</always_on>
-        <update_rate>30</update_rate>
-        <visualize>true</visualize>
+        <update_rate>15</update_rate>
+        <visualize>false</visualize>
+        <enable_metrics>false</enable_metrics>
     </sensor>
 </gazebo>
