Commit message: [Nav][Desc] modified rsp.launch.py to use sim time and modified robot.xacro

File: src/nyurdt_description/urdf/robot.xacro (robot description, xacro)
@@ -46,9 +46,9 @@
 <xacro:include filename="$(find realsense2_description)/urdf/_d435.urdf.xacro"/>
 <!-- ── Frames ─────────────────────────────────────────────────────────── -->
-<link name="base_footprint"/>
+<!-- <link name="base_footprint"/>
 <joint name="base_footprint_joint" type="fixed">
     <parent link="base_footprint"/>
     <child link="base_link"/>
-</joint>
+</joint> -->
 <!-- base_link: Nav2 + RTAB-Map reference frame, at ground centre -->
 <link name="base_link"/>

Commit message: added pitch for realsense angle

File: src/nyurdt_description/urdf/robot.xacro (robot description, xacro)
@@ -157,5 +157,5 @@
 <!-- mounted at front face centre, ~33cm off ground -->
 <xacro:sensor_d435 parent="base_link" name="camera" use_nominal_extrinsics="true">
-    <origin xyz="0.37 0.0 0.33" rpy="0 0 0"/>
+    <origin xyz="0.37 0.0 0.33" rpy="0 0.698132 0"/>
 </xacro:sensor_d435>
 <gazebo reference="camera_link">

Commit message: changes made to params to prevent slowding down over time

File: src/nyurdt_description/urdf/robot.xacro (robot description, xacro)
@@ -157,5 +157,5 @@
 <!-- mounted at front face centre, ~33cm off ground -->
 <xacro:sensor_d435 parent="base_link" name="camera" use_nominal_extrinsics="true">
-    <origin xyz="0.37 0.0 0.33" rpy="0 0.698132 0"/>
+    <origin xyz="0.37 0.0 0.33" rpy="0 0.767945 0"/>
 </xacro:sensor_d435>
 <gazebo reference="camera_link">

Commit message: Feature/rtabmap param fix (#46)
* changing params to make it run faster (realsense fps was too high)

* added pitch for realsense angle

* changes made to params to prevent slowding down over time

* remove memory limits to show all the points and trajectories

* ready to be merged

---------

Co-authored-by: andrea7308 <ag8754@nyu.edu>
Co-authored-by: MdyWg <mdywg16@gmail.com>

File: src/nyurdt_description/urdf/robot.xacro (robot description, xacro)
@@ -157,5 +157,5 @@
 <!-- mounted at front face centre, ~33cm off ground -->
 <xacro:sensor_d435 parent="base_link" name="camera" use_nominal_extrinsics="true">
-    <origin xyz="0.37 0.0 0.33" rpy="0 0 0"/>
+    <origin xyz="0.37 0.0 0.33" rpy="0 0.767945 0"/>
 </xacro:sensor_d435>
 <gazebo reference="camera_link">

Commit message: Revert "Feature/rtabmap param fix (#46)"
This reverts commit 56f160c06d994937c9ac7be1780d59c1309f95d9.

File: src/nyurdt_description/urdf/robot.xacro (robot description, xacro)
@@ -157,5 +157,5 @@
 <!-- mounted at front face centre, ~33cm off ground -->
 <xacro:sensor_d435 parent="base_link" name="camera" use_nominal_extrinsics="true">
-    <origin xyz="0.37 0.0 0.33" rpy="0 0.767945 0"/>
+    <origin xyz="0.37 0.0 0.33" rpy="0 0 0"/>
 </xacro:sensor_d435>
 <gazebo reference="camera_link">

Commit message: wip

File: src/nyurdt_description/urdf/robot.xacro (robot description, xacro)
@@ -157,5 +157,5 @@
 <!-- mounted at front face centre, ~33cm off ground -->
 <xacro:sensor_d435 parent="base_link" name="camera" use_nominal_extrinsics="true">
-    <origin xyz="0.37 0.0 0.33" rpy="0 0.767945 0"/>
+    <origin xyz="0.37 0.0 0.33" rpy="0 0.56024 0"/>
 </xacro:sensor_d435>
 <gazebo reference="camera_link">

Commit message: some stuff to try isaacross

File: src/nyurdt_description/urdf/robot.xacro (robot description, xacro)
@@ -156,11 +156,10 @@
 <!-- ── RealSense D435 ──────────────────────────────────────────────────── -->
 <!-- mounted at front face centre, ~33cm off ground -->
-<xacro:sensor_d435 parent="base_link" name="camera" use_nominal_extrinsics="true">
-    <origin xyz="0.37 0.0 0.33" rpy="0 0.56024 0"/>
+<xacro:sensor_d435 parent="base_link" name="camera0" use_nominal_extrinsics="true">
+    <origin xyz="0.37 0.0 0.33" rpy="0 0.42 0"/>
 </xacro:sensor_d435>
-<gazebo reference="camera_link">
+<gazebo reference="camera0_link">
     <sensor name="realsense_d435" type="rgbd_camera">
-        <topic>realsense</topic>
-        <camera>
+        <topic>realsense/image_raw</topic> <camera>
             <horizontal_fov>1.047</horizontal_fov>
             <image>

Commit message: switching stuff dont use

File: src/nyurdt_description/urdf/robot.xacro (robot description, xacro)
@@ -157,4 +157,5 @@
 <!-- mounted at front face centre, ~33cm off ground -->
 <xacro:sensor_d435 parent="base_link" name="camera" use_nominal_extrinsics="true">
+    <!-- <origin xyz="0.37 0.0 1.12" rpy="0 0 0"/> -->
     <origin xyz="0.37 0.0 0.33" rpy="0 0.767945 0"/>
 </xacro:sensor_d435>

Commit message: updated robot dimensions and readme to ignore pycache files

File: src/nyurdt_description/urdf/robot.xacro (robot description, xacro)
@@ -7,5 +7,5 @@
 <xacro:property name="c" value="0.660" />   <!-- height -->
 <!-- Wheel dimensions — measure and confirm these -->
-<xacro:property name="r" value="0.15" />    <!-- wheel radius -->
+<xacro:property name="r" value="0.17" />    <!-- wheel radius -->
 <xacro:property name="d" value="0.1"  />    <!-- wheel width  -->
 <xacro:property name="s1" value="${c/2}"         />   <!-- body centre height -->
@@ -46,9 +46,4 @@
 <xacro:include filename="$(find realsense2_description)/urdf/_d435.urdf.xacro"/>
 <!-- ── Frames ─────────────────────────────────────────────────────────── -->
-<!-- <link name="base_footprint"/>
-<joint name="base_footprint_joint" type="fixed">
-    <parent link="base_footprint"/>
-    <child link="base_link"/>
-</joint> -->
 <!-- base_link: Nav2 + RTAB-Map reference frame, at ground centre -->
 <link name="base_link"/>

Commit message: added cams (missing index and front cam pos)

File: src/nyurdt_description/urdf/robot.xacro (robot description, xacro)
@@ -181,3 +181,26 @@
     </sensor>
 </gazebo>
+<!-- ── Logitech C615 ──────────────────────────────────────────────────── -->
+<xacro:include filename="camera.xacro" />
+<xacro:property name="x" value=".017"/>
+<xacro:property name="y" value=".07"/>
+<xacro:property name="z" value=".04"/>
+<!-- need numbers -->
+<xacro:camera parent="base_link" pos="front" size_x="${x}" size_y="${y}" size_z="${z}">
+    <origin xyz="0 0 0" rpy="0 0 0"/>
+</xacro:camera>
+<xacro:camera parent="base_link" pos="back" size_x="${x}" size_y="${y}" size_z="${z}">
+    <origin xyz="-.2799208 -.195 .45" rpy="0 0 -${pi_const}"/>
+</xacro:camera>
+<!-- ── Innomaker ──────────────────────────────────────────────────── -->
+<xacro:include filename="camera.xacro" />
+<xacro:property name="x" value=".037"/>
+<xacro:property name="y" value=".037"/>
+<xacro:property name="z" value=".04"/>
+<xacro:camera parent="base_link" pos="right" size_x="${x}" size_y="${y}" size_z="${z}">
+    <origin xyz="0.00792 -0.195 0.45" rpy="0 0 -1.57"/>
+</xacro:camera>
+<xacro:camera parent="base_link" pos="left" size_x="${x}" size_y="${y}" size_z="${z}">
+    <origin xyz="0.00792 0.195 0.45" rpy="0 0 1.57"/>
+</xacro:camera>
 </robot>

Commit message: added front cam offset to urdf

File: src/nyurdt_description/urdf/robot.xacro (robot description, xacro)
@@ -181,7 +181,6 @@
 <xacro:property name="y" value=".07"/>
 <xacro:property name="z" value=".04"/>
-<!-- need numbers -->
 <xacro:camera parent="base_link" pos="front" size_x="${x}" size_y="${y}" size_z="${z}">
-    <origin xyz="0 0 0" rpy="0 0 0"/>
+    <origin xyz=".32792 -.195 .45" rpy="0 0 ${pi_const}"/>
 </xacro:camera>
 <xacro:camera parent="base_link" pos="back" size_x="${x}" size_y="${y}" size_z="${z}">

Commit message: attempting to get realsense stream working for rtabmap in sim

File: src/nyurdt_description/urdf/robot.xacro (robot description, xacro)
@@ -150,8 +150,4 @@
 </link>
 <!-- ── RealSense D435 ──────────────────────────────────────────────────── -->
-<!-- mounted at front face centre, ~33cm off ground -->
-<xacro:sensor_d435 parent="base_link" name="camera" use_nominal_extrinsics="true">
-    <origin xyz="0.37 0.0 0.33" rpy="0 0.767945 0"/>
-</xacro:sensor_d435>
 <gazebo reference="camera_link">
     <sensor name="realsense_d435" type="rgbd_camera">
@@ -164,5 +160,8 @@
                 <format>R8G8B8</format>
             </image>
-            <clip><near>0.1</near><far>100</far></clip>
+            <depth_camera>
+                <output>depths</output>
+            </depth_camera>
+            <clip><near>0.1</near><far>10.0</far></clip>
             <noise>
                 <type>gaussian</type>
@@ -172,5 +171,5 @@
         </camera>
         <always_on>1</always_on>
-        <update_rate>30</update_rate>
+        <update_rate>15</update_rate>
         <visualize>true</visualize>
     </sensor>

Commit message: modified deposition

File: src/nyurdt_description/urdf/robot.xacro (robot description, xacro)
@@ -152,5 +152,5 @@
 <!-- mounted at front face centre, ~33cm off ground -->
 <xacro:sensor_d435 parent="base_link" name="camera" use_nominal_extrinsics="true">
-    <origin xyz="0.37 0.0 0.78" rpy="0 0.767945 0"/>
+    <origin xyz="0.37 0.0 0.69" rpy="0 0.767945 0"/>
 </xacro:sensor_d435>
 <gazebo reference="camera_link">

Commit message: fixed deposition Duration type mismatch

File: src/nyurdt_description/urdf/robot.xacro (robot description, xacro)
@@ -152,5 +152,5 @@
 <!-- mounted at front face centre, ~33cm off ground -->
 <xacro:sensor_d435 parent="base_link" name="camera" use_nominal_extrinsics="true">
-    <origin xyz="0.37 0.0 0.33" rpy="0 0.767945 0"/>
+    <origin xyz="0.37 0.0 0.69" rpy="0 0.767945 0"/>
 </xacro:sensor_d435>
 <gazebo reference="camera_link">
